File: Taco_Raven/KiCad/ATSAMD51.sch (KiCad schematic (older format))
At the start: 31 parts, among them J1 CONN_02X05, J2 CONN_02X05, J3 CONN_01X04, J34 USB_MINI, J35 CONN_02X05, J36 CONN_02X04, SW1 SW_Push, U21 ATSAMD51, U22 SPIFLASH_SOIC8

Commit message: TMC2209 upgrade layout ready for review
Parts:
- removed J35: CONN_02X05, MZBOT:PinHeader_2x05_P1.27mm_Vertical_SMD, symbol Voron_Klipper_Board-rescue:CONN_02X05-MZBOT
- added J35: CONN_02X03, MZBOT:PinHeader_2x03_P2.54mm_Vertical, symbol MZBOT:CONN_02X03
- C115, C116, C117, C118, C119, C120, C121, C122, C123, C124, C125, C126, C127, C128: symbol Voron_Klipper_Board-rescue:C_0805-MZBOT -> MZBOT:C_0805
- J1, J2: symbol Voron_Klipper_Board-rescue:CONN_02X05-MZBOT -> MZBOT:CONN_02X05
- J3: symbol Voron_Klipper_Board-rescue:CONN_01X04-MZBOT -> MZBOT:CONN_01X04
- J34: symbol Voron_Klipper_Board-rescue:USB_MINI-MZBOT -> MZBOT:USB_MINI
- J36: symbol Voron_Klipper_Board-rescue:CONN_02X04-MZBOT -> MZBOT:CONN_02X04
- L1: symbol Voron_Klipper_Board-rescue:Inductor-MZBOT -> MZBOT:Inductor
- L2: symbol Voron_Klipper_Board-rescue:Ferrite_0805-MZBOT -> MZBOT:Ferrite_0805
- R91, R92, R93, R97, R98, R99: symbol Voron_Klipper_Board-rescue:R_0805-MZBOT -> MZBOT:R_0805
- SW1: symbol Voron_Klipper_Board-rescue:SW_Push-MZBOT -> MZBOT:SW_Push
- U21: symbol Voron_Klipper_Board-rescue:SAM51-MZBOT -> MZBOT:SAM51
- U22: symbol Voron_Klipper_Board-rescue:SPIFLASH_SOIC8-MZBOT -> MZBOT:SPIFLASH_SOIC8
Connections:
- net labels added: KILL, RRFGD_LCD5, RRFGD_LCD6, RRFGD_LCD7, TMC_UART0, TMC_UART1
- net labels removed: SPI_CS_E0, SPI_CS_E1, SPI_CS_X, SPI_CS_Y, SPI_CS_Z0, SPI_CS_Z1, SPI_CS_Z2, SPI_CS_Z3
- wire segments 260 -> 261
Other:
- note added: "TCC(3.0)(0.4) {Still Valid?}"
- note added: "TCC0.6"
- note added: "TCC1.0\n"
- note added: "TCC1.3"
- note added: "{Still Valid?} TCC1.3\n"
- note removed: "TCC(3.0)(0.4)"
- note removed: "TCC(3.1)(0.5)"
- note removed: "TCC1.0"
- note removed: "TCC1.1"
- note removed: "TCC1.3\n"
