File: Taco_Raven/KiCad/Endstops.sch (KiCad schematic (older format))
At the start: 26 parts, among them J29 CONN_01X03, J30 CONN_01X03, J31 CONN_01X03, J32 CONN_01X03, J33 CONN_01X03

Commit message: TMC2209 upgrade layout ready for review
Parts:
- C134, C135, C136, C137, C138: symbol Voron_Klipper_Board-rescue:C_0805-MZBOT -> MZBOT:C_0805
- D10, D5, D6, D7, D8: symbol Voron_Klipper_Board-rescue:LED_0805-MZBOT -> MZBOT:LED_0805
- D9: symbol Voron_Klipper_Board-rescue:BAT43-MZBOT -> MZBOT:BAT43
- J29, J30, J31, J32, J33: symbol Voron_Klipper_Board-rescue:CONN_01X03-MZBOT -> MZBOT:CONN_01X03
- R65, R66, R67, R68, R69, R70, R71, R72, R73, R74: symbol Voron_Klipper_Board-rescue:R_0805-MZBOT -> MZBOT:R_0805
Changed lines of the file:
@@
 Connection ~ 3125 2775
 $Comp
-L Voron_Klipper_Board-rescue:GND-MZBOT #PWR?
+L MZBOT:GND #PWR?
 U 1 1 5BA95C31
 P 3125 3225
@@
 	3125 3175 3125 3225
 $Comp
-L Voron_Klipper_Board-rescue:+3.3V-MZBOT #PWR0134
+L MZBOT:+3.3V #PWR0134
 U 1 1 5BA964D6
 P 3650 1950
@@
 	3650 1950 3650 2025
 $Comp
-L Voron_Klipper_Board-rescue:CONN_01X03-MZBOT J29
+L MZBOT:CONN_01X03 J29
 U 1 1 5BA9732D
 P 4150 2875
@@
 	3900 2875 3900 2700
 $Comp
-L Voron_Klipper_Board-rescue:+3.3V-MZBOT #PWR0136
+L MZBOT:+3.3V #PWR0136
 U 1 1 5BA97660
 P 3900 2700
@@
 	3900 2975 3900 3125
 $Comp
-L Voron_Klipper_Board-rescue:GND-MZBOT #PWR?
+L MZBOT:GND #PWR?
 U 1 1 5BA97813
 P 3900 3125
@@
 Connection ~ 5275 2775
 $Comp
-L Voron_Klipper_Board-rescue:GND-MZBOT #PWR?
+L MZBOT:GND #PWR?
 U 1 1 5BA9C3A8
 P 5275 3225
@@
 	5275 3175 5275 3225
 $Comp
-L Voron_Klipper_Board-rescue:+3.3V-MZBOT #PWR0142
+L MZBOT:+3.3V #PWR0142
 U 1 1 5BA9C3B6
 P 5800 1950
@@
 	6275 2975 6275 3125
 $Comp
-L Voron_Klipper_Board-rescue:GND-MZBOT #PWR?
+L MZBOT:GND #PWR?
 U 1 1 5BA9C3CF
 P 6275 3125
@@
 Connection ~ 7625 2775
 $Comp
-L Voron_Klipper_Board-rescue:GND-MZBOT #PWR?
+L MZBOT:GND #PWR?
 U 1 1 5BA9C6CA
 P 7625 3225
@@
 	7625 3175 7625 3225
 $Comp
-L Voron_Klipper_Board-rescue:+3.3V-MZBOT #PWR0149
+L MZBOT:+3.3V #PWR0149
 U 1 1 5BA9C6D8
 P 8150 1950
@@
 	8400 2875 8400 2700
 $Comp
-L Voron_Klipper_Board-rescue:+3.3V-MZBOT #PWR0150
+L MZBOT:+3.3V #PWR0150
 U 1 1 5BA9C6E9
 P 8400 2700
@@
 	8400 2975 8400 3125
 $Comp
-L Voron_Klipper_Board-rescue:GND-MZBOT #PWR?
+L MZBOT:GND #PWR?
 U 1 1 5BA9C6F1
 P 8400 3125
@@
 Connection ~ 3125 5000
 $Comp
-L Voron_Klipper_Board-rescue:GND-MZBOT #PWR?
+L MZBOT:GND #PWR?
 U 1 1 5BA9CCFE
 P 3125 5450
@@
 	3125 5400 3125 5450
 $Comp
-L Voron_Klipper_Board-rescue:+3.3V-MZBOT #PWR0135
+L MZBOT:+3.3V #PWR0135
 U 1 1 5BA9CD0C
 P 3650 4175
@@
 	3900 5100 3900 4925
 $Comp
-L Voron_Klipper_Board-rescue:+3.3V-MZBOT #PWR0138
+L MZBOT:+3.3V #PWR0138
 U 1 1 5BA9CD1D
 P 3900 4925
@@
 	3900 5200 3900 5350
 $Comp
-L Voron_Klipper_Board-rescue:GND-MZBOT #PWR?
+L MZBOT:GND #PWR?
 U 1 1 5BA9CD25
 P 3900 5350
@@
 Connection ~ 5375 5000
 $Comp
-L Voron_Klipper_Board-rescue:GND-MZBOT #PWR?
+L MZBOT:GND #PWR?
 U 1 1 5BA9D8D1
 P 5375 5450
@@
 	5375 5400 5375 5450
 $Comp
-L Voron_Klipper_Board-rescue:+3.3V-MZBOT #PWR0143
+L MZBOT:+3.3V #PWR0143
 U 1 1 5BA9D8DF
 P 5900 4175
@@
 	6150 5100 6150 4925
 $Comp
-L Voron_Klipper_Board-rescue:+3.3V-MZBOT #PWR0144
+L MZBOT:+3.3V #PWR0144
 U 1 1 5BA9D8F0
 P 6150 4925
@@
 	6150 5200 6150 5350
 $Comp
-L Voron_Klipper_Board-rescue:GND-MZBOT #PWR?
+L MZBOT:GND #PWR?
 U 1 1 5BA9D8F8
 P 6150 5350
@@
 NPN Inductive\nsensors only
 $Comp
-L Voron_Klipper_Board-rescue:+12V-MZBOT #PWR0146
+L MZBOT:+12V #PWR0146
 U 1 1 5C2DC5A9
 P 6275 2700
@@
 ENDSTOP_E1
 $Comp
-L Voron_Klipper_Board-rescue:BAT43-MZBOT D9
+L MZBOT:BAT43 D9
 U 1 1 5C12FEF0
 P 6025 2775
@@
 $EndComp
 $Comp
-L Voron_Klipper_Board-rescue:R_0805-MZBOT R?
+L MZBOT:R_0805 R?
 U 1 1 608289D6
 P 3400 2775
@@
 $EndComp
 $Comp
-L Voron_Klipper_Board-rescue:R_0805-MZBOT R?
+L MZBOT:R_0805 R?
 U 1 1 6082AFAA
 P 5550 2775
@@
 $EndComp
 $Comp
-L Voron_Klipper_Board-rescue:R_0805-MZBOT R?
+L MZBOT:R_0805 R?
 U 1 1 6082B17A
 P 7900 2775
@@
 $EndComp
 $Comp
-L Voron_Klipper_Board-rescue:R_0805-MZBOT R?
+L MZBOT:R_0805 R?
 U 1 1 6082B214
 P 5650 5000
@@
 $EndComp
 $Comp
-L Voron_Klipper_Board-rescue:R_0805-MZBOT R?
+L MZBOT:R_0805 R?
 U 1 1 6082B42A
 P 3400 5000
@@
 $EndComp
 $Comp
-L Voron_Klipper_Board-rescue:C_0805-MZBOT C?
+L MZBOT:C_0805 C?
 U 1 1 6082C5E8
 P 3125 3025
@@
 $EndComp
 $Comp
-L Voron_Klipper_Board-rescue:C_0805-MZBOT C?
+L MZBOT:C_0805 C?
 U 1 1 6082D9A9
 P 5275 3025
@@
 $EndComp
 $Comp
-L Voron_Klipper_Board-rescue:C_0805-MZBOT C?
+L MZBOT:C_0805 C?
 U 1 1 6082DBBB
 P 7625 3025
@@
 $EndComp
 $Comp
-L Voron_Klipper_Board-rescue:C_0805-MZBOT C?
+L MZBOT:C_0805 C?
 U 1 1 6082DC77
 P 5375 5250
@@
 $EndComp
 $Comp
-L Voron_Klipper_Board-rescue:C_0805-MZBOT C?
+L MZBOT:C_0805 C?
 U 1 1 6082DE65
 P 3125 5250
@@
 $EndComp
 $Comp
-L Voron_Klipper_Board-rescue:R_0805-MZBOT R?
+L MZBOT:R_0805 R?
 U 1 1 6082EB97
 P 3650 2175
@@
 $EndComp
 $Comp
-L Voron_Klipper_Board-rescue:R_0805-MZBOT R?
+L MZBOT:R_0805 R?
 U 1 1 60830360
 P 5800 2175
@@
 $EndComp
 $Comp
-L Voron_Klipper_Board-rescue:R_0805-MZBOT R?
+L MZBOT:R_0805 R?
 U 1 1 608303E8
 P 8150 2175
@@
 $EndComp
 $Comp
-L Voron_Klipper_Board-rescue:R_0805-MZBOT R?
+L MZBOT:R_0805 R?
 U 1 1 60830581
 P 5900 4400
@@
 $EndComp
 $Comp
-L Voron_Klipper_Board-rescue:R_0805-MZBOT R?
+L MZBOT:R_0805 R?
 U 1 1 60830763
 P 3650 4400
@@
 $EndComp
 $Comp
-L Voron_Klipper_Board-rescue:LED_0805-MZBOT D?
+L MZBOT:LED_0805 D?
 U 1 1 60831941
 P 3650 2550
@@
 $EndComp
 $Comp
-L Voron_Klipper_Board-rescue:LED_0805-MZBOT D?
+L MZBOT:LED_0805 D?
 U 1 1 60832B02
 P 5800 2550
@@
 $EndComp
 $Comp
-L Voron_Klipper_Board-rescue:LED_0805-MZBOT D?
+L MZBOT:LED_0805 D?
 U 1 1 60832C1A
 P 8150 2550
@@
 $EndComp
 $Comp
-L Voron_Klipper_Board-rescue:LED_0805-MZBOT D?
+L MZBOT:LED_0805 D?
 U 1 1 60832DF4
 P 5900 4775
@@
 $EndComp
 $Comp
-L Voron_Klipper_Board-rescue:LED_0805-MZBOT D?
+L MZBOT:LED_0805 D?
 U 1 1 60832FFB
 P 3650 4775
@@
 $EndComp
 $Comp
-L Voron_Klipper_Board-rescue:CONN_01X03-MZBOT J32
+L MZBOT:CONN_01X03 J32
 U 1 1 6083467C
 P 6525 2875
@@
 $EndComp
 $Comp
-L Voron_Klipper_Board-rescue:CONN_01X03-MZBOT J33
+L MZBOT:CONN_01X03 J33
 U 1 1 60834849
 P 8650 2875
@@
 $EndComp
 $Comp
-L Voron_Klipper_Board-rescue:CONN_01X03-MZBOT J31
+L MZBOT:CONN_01X03 J31
 U 1 1 60834A6F
 P 6400 5100
@@
 $EndComp
 $Comp
-L Voron_Klipper_Board-rescue:CONN_01X03-MZBOT J30
+L MZBOT:CONN_01X03 J30
 U 1 1 60834BD2
 P 4150 5100
