File: Taco_Raven/KiCad/FANS.sch (KiCad schematic (older format))
At the start: 23 parts, among them J12 CONN_02X03, J13 CONN_01X02, J14 CONN_01X02, J15 CONN_01X02, J16 CONN_01X02, J17 CONN_01X02, J18 CONN_01X02, J19 CONN_01X02, U10 PMV40UN, U11 PMV40UN, U12 PMV40UN, U13 PMV40UN, U9 PMV40UN

Commit message: TMC2209 upgrade layout ready for review
Parts:
- J12: symbol Voron_Klipper_Board-rescue:CONN_02X03-MZBOT -> MZBOT:CONN_02X03
- J13, J14, J15, J16, J17, J18, J19: symbol Voron_Klipper_Board-rescue:CONN_01X02-MZBOT -> MZBOT:CONN_01X02
- R33, R34, R35, R36, R37, R38, R39, R40, R41, R42: symbol Voron_Klipper_Board-rescue:R_0805-MZBOT -> MZBOT:R_0805
- U10, U11, U12, U13, U9: symbol Voron_Klipper_Board-rescue:PMV40UN-MZBOT -> MZBOT:PMV40UN
Changed lines of the file:
@@
 $EndDescr
 $Comp
-L Voron_Klipper_Board-rescue:CONN_01X02-MZBOT J13
+L MZBOT:CONN_01X02 J13
 U 1 1 5BB756A0
 P 4550 2050
@@
 $EndComp
 $Comp
-L Voron_Klipper_Board-rescue:PMV40UN-MZBOT U9
+L MZBOT:PMV40UN U9
 U 1 1 5BB771FB
 P 4250 2400
@@
 	4250 2000 4250 1875
 $Comp
-L Voron_Klipper_Board-rescue:+V_FAN-MZBOT #PWR098
+L MZBOT:+V_FAN #PWR098
 U 1 1 5BB79357
 P 4250 1875
@@
 $EndComp
 $Comp
-L Voron_Klipper_Board-rescue:GND-MZBOT #PWR?
+L MZBOT:GND #PWR?
 U 1 1 5BB794EF
 P 4250 2700
@@
 	3900 2400 3950 2400
 $Comp
-L Voron_Klipper_Board-rescue:GND-MZBOT #PWR?
+L MZBOT:GND #PWR?
 U 1 1 5BB7D4A7
 P 3500 2850
@@
 	6700 2000 6700 1875
 $Comp
-L Voron_Klipper_Board-rescue:+V_FAN-MZBOT #PWR0104
+L MZBOT:+V_FAN #PWR0104
 U 1 1 5BB82FD8
 P 6700 1875
@@
 $EndComp
 $Comp
-L Voron_Klipper_Board-rescue:GND-MZBOT #PWR?
+L MZBOT:GND #PWR?
 U 1 1 5BB82FDE
 P 6700 2700
@@
 	6350 2400 6400 2400
 $Comp
-L Voron_Klipper_Board-rescue:GND-MZBOT #PWR?
+L MZBOT:GND #PWR?
 U 1 1 5BB82FFE
 P 5950 2850
@@
 	9150 2000 9150 1875
 $Comp
-L Voron_Klipper_Board-rescue:+V_FAN-MZBOT #PWR0113
+L MZBOT:+V_FAN #PWR0113
 U 1 1 5BB83250
 P 9150 1875
@@
 $EndComp
 $Comp
-L Voron_Klipper_Board-rescue:GND-MZBOT #PWR?
+L MZBOT:GND #PWR?
 U 1 1 5BB83256
 P 9150 2700
@@
 	8800 2400 8850 2400
 $Comp
-L Voron_Klipper_Board-rescue:GND-MZBOT #PWR?
+L MZBOT:GND #PWR?
 U 1 1 5BB83276
 P 8400 2850
@@
 	4250 4400 4250 4275
 $Comp
-L Voron_Klipper_Board-rescue:+V_FAN-MZBOT #PWR0100
+L MZBOT:+V_FAN #PWR0100
 U 1 1 5BB83722
 P 4250 4275
@@
 $EndComp
 $Comp
-L Voron_Klipper_Board-rescue:GND-MZBOT #PWR?
+L MZBOT:GND #PWR?
 U 1 1 5BB83728
 P 4250 5100
@@
 	3900 4800 3950 4800
 $Comp
-L Voron_Klipper_Board-rescue:GND-MZBOT #PWR?
+L MZBOT:GND #PWR?
 U 1 1 5BB83748
 P 3500 5250
@@
 	6700 4400 6700 4275
 $Comp
-L Voron_Klipper_Board-rescue:+V_FAN-MZBOT #PWR0106
+L MZBOT:+V_FAN #PWR0106
 U 1 1 5BB83EC7
 P 6700 4275
@@
 $EndComp
 $Comp
-L Voron_Klipper_Board-rescue:GND-MZBOT #PWR?
+L MZBOT:GND #PWR?
 U 1 1 5BB83ECD
 P 6700 5100
@@
 	6350 4800 6400 4800
 $Comp
-L Voron_Klipper_Board-rescue:GND-MZBOT #PWR?
+L MZBOT:GND #PWR?
 U 1 1 5BB83EED
 P 5950 5250
@@
 	9125 4725 9125 4600
 $Comp
-L Voron_Klipper_Board-rescue:+V_FAN-MZBOT #PWR0111
+L MZBOT:+V_FAN #PWR0111
 U 1 1 5BB85F08
 P 9125 4600
@@
 	7975 4725 7975 4600
 $Comp
-L Voron_Klipper_Board-rescue:+V_FAN-MZBOT #PWR0108
+L MZBOT:+V_FAN #PWR0108
 U 1 1 5BB8719D
 P 7975 4600
@@
 $EndComp
 $Comp
-L Voron_Klipper_Board-rescue:GND-MZBOT #PWR?
+L MZBOT:GND #PWR?
 U 1 1 5BB9519A
 P 7975 4900
@@
 	7975 4825 7975 4900
 $Comp
-L Voron_Klipper_Board-rescue:GND-MZBOT #PWR?
+L MZBOT:GND #PWR?
 U 1 1 5BB95F02
 P 9125 4900
@@
 ALWAYS ON FANS
 $Comp
-L Voron_Klipper_Board-rescue:+12V-MZBOT #PWR093
+L MZBOT:+12V #PWR093
 U 1 1 5BCD4B04
 P 1700 1950
@@
 $EndComp
 $Comp
-L Voron_Klipper_Board-rescue:+5V-MZBOT #PWR094
+L MZBOT:+5V #PWR094
 U 1 1 5BCD4B5B
 P 1600 1850
@@
 FAN0
 $Comp
-L Voron_Klipper_Board-rescue:CONN_02X03-MZBOT J12
+L MZBOT:CONN_02X03 J12
 U 1 1 5CE033A6
 P 1700 2300
@@
 	1800 2050 1800 2100
 $Comp
-L Voron_Klipper_Board-rescue:+V_FAN-MZBOT #PWR095
+L MZBOT:+V_FAN #PWR095
 U 1 1 5BCD0145
 P 2000 2750
@@
 	1800 2800 1700 2800
 $Comp
-L Voron_Klipper_Board-rescue:+VIN_FUSED-MZBOT #PWR0196
+L MZBOT:+VIN_FUSED #PWR0196
 U 1 1 5CE125EE
 P 1800 2050
@@
 $EndComp
 $Comp
-L Voron_Klipper_Board-rescue:R_0805-MZBOT R?
+L MZBOT:R_0805 R?
 U 1 1 607F7894
 P 3500 2625
@@
 $EndComp
 $Comp
-L Voron_Klipper_Board-rescue:R_0805-MZBOT R?
+L MZBOT:R_0805 R?
 U 1 1 607F8EF8
 P 5950 2625
@@
 $EndComp
 $Comp
-L Voron_Klipper_Board-rescue:R_0805-MZBOT R?
+L MZBOT:R_0805 R?
 U 1 1 607F8F5C
 P 8400 2625
@@
 $EndComp
 $Comp
-L Voron_Klipper_Board-rescue:R_0805-MZBOT R?
+L MZBOT:R_0805 R?
 U 1 1 607F9003
 P 5950 5025
@@
 $EndComp
 $Comp
-L Voron_Klipper_Board-rescue:R_0805-MZBOT R?
+L MZBOT:R_0805 R?
 U 1 1 607F9137
 P 3500 5025
@@
 $EndComp
 $Comp
-L Voron_Klipper_Board-rescue:R_0805-MZBOT R?
+L MZBOT:R_0805 R?
 U 1 1 607F9848
 P 3750 2400
@@
 $EndComp
 $Comp
-L Voron_Klipper_Board-rescue:R_0805-MZBOT R?
+L MZBOT:R_0805 R?
 U 1 1 607FB03C
 P 6200 2400
@@
 $EndComp
 $Comp
-L Voron_Klipper_Board-rescue:R_0805-MZBOT R?
+L MZBOT:R_0805 R?
 U 1 1 607FB0E6
 P 3750 4800
@@
 $EndComp
 $Comp
-L Voron_Klipper_Board-rescue:R_0805-MZBOT R?
+L MZBOT:R_0805 R?
 U 1 1 607FB276
 P 6200 4800
@@
 $EndComp
 $Comp
-L Voron_Klipper_Board-rescue:R_0805-MZBOT R?
+L MZBOT:R_0805 R?
 U 1 1 607FB37C
 P 8650 2400
@@
 $EndComp
 $Comp
-L Voron_Klipper_Board-rescue:PMV40UN-MZBOT U11
+L MZBOT:PMV40UN U11
 U 1 1 607FC001
 P 6700 2400
@@
 $EndComp
 $Comp
-L Voron_Klipper_Board-rescue:PMV40UN-MZBOT U13
+L MZBOT:PMV40UN U13
 U 1 1 607FC0B3
 P 9150 2400
@@
 $EndComp
 $Comp
-L Voron_Klipper_Board-rescue:PMV40UN-MZBOT U12
+L MZBOT:PMV40UN U12
 U 1 1 607FC123
 P 6700 4800
@@
 $EndComp
 $Comp
-L Voron_Klipper_Board-rescue:PMV40UN-MZBOT U10
+L MZBOT:PMV40UN U10
 U 1 1 607FC1A7
 P 4250 4800
@@
 $EndComp
 $Comp
-L Voron_Klipper_Board-rescue:CONN_01X02-MZBOT J15
+L MZBOT:CONN_01X02 J15
 U 1 1 607FCD33
 P 7000 2050
@@
 $EndComp
 $Comp
-L Voron_Klipper_Board-rescue:CONN_01X02-MZBOT J19
+L MZBOT:CONN_01X02 J19
 U 1 1 607FCD8B
 P 9450 2050
@@
 $EndComp
 $Comp
-L Voron_Klipper_Board-rescue:CONN_01X02-MZBOT J18
+L MZBOT:CONN_01X02 J18
 U 1 1 607FCE66
 P 9425 4775
@@
 $EndComp
 $Comp
-L Voron_Klipper_Board-rescue:CONN_01X02-MZBOT J17
+L MZBOT:CONN_01X02 J17
 U 1 1 607FCEE2
 P 8275 4775
@@
 $EndComp
 $Comp
-L Voron_Klipper_Board-rescue:CONN_01X02-MZBOT J16
+L MZBOT:CONN_01X02 J16
 U 1 1 607FCF60
 P 7000 4450
@@
 $EndComp
 $Comp
-L Voron_Klipper_Board-rescue:CONN_01X02-MZBOT J14
+L MZBOT:CONN_01X02 J14
 U 1 1 607FCFD8
 P 4550 4450
