File: Taco_Raven/KiCad/Heaters.sch (KiCad schematic (older format))
At the start: 23 parts, among them J26 CONN_01X02, J27 CONN_01X02, J28 CONN_01X02, U14 CSD18532, U15 CSD18532, U16 CSD18532, U17 CSD18532

Commit message: TMC2209 upgrade layout ready for review
Parts:
- D1, D2, D3, D4: symbol Voron_Klipper_Board-rescue:LED_0805-MZBOT -> MZBOT:LED_0805
- J26, J27, J28: symbol Voron_Klipper_Board-rescue:CONN_01X02-MZBOT -> MZBOT:CONN_01X02
- R53, R54, R55, R56, R57, R58, R59, R60, R61, R62, R63, R64: symbol Voron_Klipper_Board-rescue:R_0805-MZBOT -> MZBOT:R_0805
- U14, U15, U16, U17: symbol Voron_Klipper_Board-rescue:CSD18532-MZBOT -> MZBOT:CSD18532
Changed lines of the file:
@@
 	4400 2050 4500 2050
 $Comp
-L Voron_Klipper_Board-rescue:GND-MZBOT #PWR?
+L MZBOT:GND #PWR?
 U 1 1 5BF877DF
 P 4400 2650
@@
 	4050 2350 4100 2350
 $Comp
-L Voron_Klipper_Board-rescue:GND-MZBOT #PWR?
+L MZBOT:GND #PWR?
 U 1 1 5BF877FF
 P 3650 2800
@@
 BED\n
 $Comp
-L Voron_Klipper_Board-rescue:VBED_FUSED-MZBOT #PWR0122
+L MZBOT:VBED_FUSED #PWR0122
 U 1 1 5C0BD4A7
 P 4150 1450
@@
 	4400 4200 4400 3750
 $Comp
-L Voron_Klipper_Board-rescue:GND-MZBOT #PWR?
+L MZBOT:GND #PWR?
 U 1 1 5C0C2DD4
 P 4400 4900
@@
 	4050 4600 4100 4600
 $Comp
-L Voron_Klipper_Board-rescue:GND-MZBOT #PWR?
+L MZBOT:GND #PWR?
 U 1 1 5C0C2DF4
 P 3650 5050
@@
 	7375 1950 7375 1500
 $Comp
-L Voron_Klipper_Board-rescue:GND-MZBOT #PWR?
+L MZBOT:GND #PWR?
 U 1 1 5C0C33D8
 P 7375 2650
@@
 	7025 2350 7075 2350
 $Comp
-L Voron_Klipper_Board-rescue:GND-MZBOT #PWR?
+L MZBOT:GND #PWR?
 U 1 1 5C0C33F8
 P 6625 2800
@@
 	7375 4200 7375 3750
 $Comp
-L Voron_Klipper_Board-rescue:GND-MZBOT #PWR?
+L MZBOT:GND #PWR?
 U 1 1 5C0C3EC6
 P 7375 4900
@@
 	7025 4600 7075 4600
 $Comp
-L Voron_Klipper_Board-rescue:GND-MZBOT #PWR?
+L MZBOT:GND #PWR?
 U 1 1 5C0C3EE6
 P 6625 5050
@@
 	7375 3750 7375 3725
 $Comp
-L Voron_Klipper_Board-rescue:+VIN_FUSED-MZBOT #PWR0128
+L MZBOT:+VIN_FUSED #PWR0128
 U 1 1 5C0C78C1
 P 7375 1475
@@
 $EndComp
 $Comp
-L Voron_Klipper_Board-rescue:+VIN_FUSED-MZBOT #PWR0124
+L MZBOT:+VIN_FUSED #PWR0124
 U 1 1 5C0C79DA
 P 4400 3725
@@
 $EndComp
 $Comp
-L Voron_Klipper_Board-rescue:+VIN_FUSED-MZBOT #PWR0130
+L MZBOT:+VIN_FUSED #PWR0130
 U 1 1 5C0C7B0B
 P 7375 3725
@@
 BED
 $Comp
-L Voron_Klipper_Board-rescue:LED_0805-MZBOT D3
+L MZBOT:LED_0805 D3
 U 1 1 60812199
 P 7125 1975
@@
 $EndComp
 $Comp
-L Voron_Klipper_Board-rescue:LED_0805-MZBOT D4
+L MZBOT:LED_0805 D4
 U 1 1 608122E5
 P 7125 4225
@@
 $EndComp
 $Comp
-L Voron_Klipper_Board-rescue:LED_0805-MZBOT D2
+L MZBOT:LED_0805 D2
 U 1 1 6081238D
 P 4150 4225
@@
 $EndComp
 $Comp
-L Voron_Klipper_Board-rescue:CONN_01X02-MZBOT J?
+L MZBOT:CONN_01X02 J?
 U 1 1 60814740
 P 7675 2000
@@
 $EndComp
 $Comp
-L Voron_Klipper_Board-rescue:CSD18532-MZBOT U14
+L MZBOT:CSD18532 U14
 U 1 1 60819357
 P 4400 2350
@@
 $EndComp
 $Comp
-L Voron_Klipper_Board-rescue:CSD18532-MZBOT U15
+L MZBOT:CSD18532 U15
 U 1 1 60819685
 P 4400 4600
@@
 $EndComp
 $Comp
-L Voron_Klipper_Board-rescue:CSD18532-MZBOT U17
+L MZBOT:CSD18532 U17
 U 1 1 6081981F
 P 7375 4600
@@
 $EndComp
 $Comp
-L Voron_Klipper_Board-rescue:R_0805-MZBOT R?
+L MZBOT:R_0805 R?
 U 1 1 6081A889
 P 3650 2575
@@
 $EndComp
 $Comp
-L Voron_Klipper_Board-rescue:R_0805-MZBOT R?
+L MZBOT:R_0805 R?
 U 1 1 6081B83C
 P 6625 2575
@@
 $EndComp
 $Comp
-L Voron_Klipper_Board-rescue:R_0805-MZBOT R?
+L MZBOT:R_0805 R?
 U 1 1 6081BA7A
 P 6625 4825
@@
 $EndComp
 $Comp
-L Voron_Klipper_Board-rescue:R_0805-MZBOT R?
+L MZBOT:R_0805 R?
 U 1 1 6081BB72
 P 3650 4825
@@
 $EndComp
 $Comp
-L Voron_Klipper_Board-rescue:R_0805-MZBOT R?
+L MZBOT:R_0805 R?
 U 1 1 6081CAC9
 P 3900 2350
@@
 $EndComp
 $Comp
-L Voron_Klipper_Board-rescue:R_0805-MZBOT R?
+L MZBOT:R_0805 R?
 U 1 1 60821BA2
 P 6875 2350
@@
 $EndComp
 $Comp
-L Voron_Klipper_Board-rescue:R_0805-MZBOT R?
+L MZBOT:R_0805 R?
 U 1 1 60821E09
 P 6875 4600
@@
 $EndComp
 $Comp
-L Voron_Klipper_Board-rescue:R_0805-MZBOT R?
+L MZBOT:R_0805 R?
 U 1 1 60821F9D
 P 3900 4600
@@
 $EndComp
 $Comp
-L Voron_Klipper_Board-rescue:R_0805-MZBOT R?
+L MZBOT:R_0805 R?
 U 1 1 60825021
 P 4150 3950
@@
 $EndComp
 $Comp
-L Voron_Klipper_Board-rescue:R_0805-MZBOT R?
+L MZBOT:R_0805 R?
 U 1 1 60825641
 P 7125 1700
@@
 $EndComp
 $Comp
-L Voron_Klipper_Board-rescue:R_0805-MZBOT R?
+L MZBOT:R_0805 R?
 U 1 1 608257CE
 P 7125 3950
@@
 $EndComp
 $Comp
-L Voron_Klipper_Board-rescue:R_0805-MZBOT R?
+L MZBOT:R_0805 R?
 U 1 1 608255F3
 P 4150 1700
@@
 	4150 1875 4150 1850
 $Comp
-L Voron_Klipper_Board-rescue:LED_0805-MZBOT D1
+L MZBOT:LED_0805 D1
 U 1 1 5C0BD71B
 P 4150 1975
@@
 $EndComp
 $Comp
-L Voron_Klipper_Board-rescue:CSD18532-MZBOT U16
+L MZBOT:CSD18532 U16
 U 1 1 60A2CFC2
 P 7375 2350
@@
 $EndComp
 $Comp
-L Voron_Klipper_Board-rescue:CONN_01X02-MZBOT J?
+L MZBOT:CONN_01X02 J?
 U 1 1 5E8EED72
 P 7675 4250
@@
 $EndComp
 $Comp
-L Voron_Klipper_Board-rescue:CONN_01X02-MZBOT J?
+L MZBOT:CONN_01X02 J?
 U 1 1 5E8EEEC2
 P 4700 4250
