File: Taco_Raven/KiCad/Power.sch (KiCad schematic (older format))
At the start: 66 parts, among them J25 CONN_01X06, U18 AP2112-3.3, U19 A4403, U20 A4403, U23 PMV40UN

Commit message: TMC2209 upgrade layout ready for review
Parts:
- C113, C114, C139, C140, C141, C142, C143, C144, C145, C146, C147, C148, C153, C154, C155, C156, C157, C158, C163, C164: symbol Voron_Klipper_Board-rescue:C_0805-MZBOT -> MZBOT:C_0805
- C149, C150: symbol Voron_Klipper_Board-rescue:CP1-MZBOT -> MZBOT:CP1
- C151, C152, C159, C160, C161, C162: symbol Voron_Klipper_Board-rescue:C_1210-MZBOT -> MZBOT:C_1210
- D11, D12, D13, D14: symbol Voron_Klipper_Board-rescue:LED_0805-MZBOT -> MZBOT:LED_0805
- D15, D16, D17, D18, D19: symbol Voron_Klipper_Board-rescue:DB2W40300L-MZBOT -> MZBOT:DB2W40300L
- F1, F2, F3: symbol Voron_Klipper_Board-rescue:Fuse_Holder-MZBOT -> MZBOT:Fuse_Holder
- J25: symbol Voron_Klipper_Board-rescue:CONN_01X06-MZBOT -> MZBOT:CONN_01X06
- L3, L4: symbol Voron_Klipper_Board-rescue:Inductor-MZBOT -> MZBOT:Inductor
- R75, R76, R77, R78, R79, R80, R81, R82, R87, R88, R89, R90, R94, R95, R96: symbol Voron_Klipper_Board-rescue:R_0805-MZBOT -> MZBOT:R_0805
- R83, R84, R85, R86: symbol Voron_Klipper_Board-rescue:R_1210-MZBOT -> MZBOT:R_1210
- U18: symbol Voron_Klipper_Board-rescue:AP2112-3.3-MZBOT -> MZBOT:AP2112-3.3
- U19, U20: symbol Voron_Klipper_Board-rescue:A4403-MZBOT -> MZBOT:A4403
- U23: symbol Voron_Klipper_Board-rescue:PMV40UN-MZBOT -> MZBOT:PMV40UN
Connections:
- no-connect marks 0 -> 1
