File: Taco_Raven/KiCad/StepperXYE0E1.sch (KiCad schematic (older format))
At the start: 80 parts, among them J4 CONN_01X04, J5 CONN_01X04, J6 CONN_01X04, J7 CONN_01X04, U1 TMC2130, U2 TMC2130, U3 TMC2130, U4 TMC2130

Commit message: TMC2209 upgrade layout ready for review
Parts:
- removed C3, C30, C32, C33, C34, C35, C36, C4, C5, C6, C7, C8: 100nF, MZBOT:C_0603, symbol Voron_Klipper_Board-rescue:C_0805-MZBOT
- removed R1, R10, R2, R9: 10.0K, MZBOT:R_0603, symbol Voron_Klipper_Board-rescue:R_0805-MZBOT
- removed R11, R12, R3, R4: 10R, MZBOT:R_0603, symbol Voron_Klipper_Board-rescue:R_0805-MZBOT
- removed U1, U2, U3, U4: TMC2130, MZBOT:QFN36_0.5_5.0X6.0, symbol Voron_Klipper_Board-rescue:TMC2130-MZBOT
- added C3, C32, C5, C8: 4.7uF, MZBOT:C_0805, symbol MZBOT:C_0805
- added C30, C4, C6, C7: 100nF, MZBOT:C_0603, symbol MZBOT:C_0805
- added R1, R2, R3: 10.0K, MZBOT:R_0603, symbol MZBOT:R_0805
- added U1, U2, U3, U4: TMC2209, MZBOT:QFN-28_EP_5x5_Pitch0.5mm, symbol MZBOT:TMC2209
- C1, C10, C11, C12, C13, C14, C15, C16, C17, C18, C19, C2, C20, C21, C23, C24, C25, C26, C27, C28, C29, C37, C38, C39, C40, C41, C42, C43, C44, C45, C46, C47, C48, C49, C50, C52, C54, C55, C56, C9: symbol Voron_Klipper_Board-rescue:C_0805-MZBOT -> MZBOT:C_0805
- C22, C31, C51, C53: symbol Voron_Klipper_Board-rescue:CP1-MZBOT -> MZBOT:CP1
- J4, J5, J6, J7: symbol Voron_Klipper_Board-rescue:CONN_01X04-MZBOT -> MZBOT:CONN_01X04
- R13, R14, R15, R16, R5, R6, R7, R8: symbol Voron_Klipper_Board-rescue:R_0805-MZBOT -> MZBOT:R_0805
Connections:
- net labels added: TMC_UART0
- net labels removed: +5V, SPI_CLK, SPI_CS_E0, SPI_CS_E1, SPI_CS_X, SPI_CS_Y, SPI_SDI, SPI_SDO
- wire segments 512 -> 360
- no-connect marks 0 -> 12
