File: Taco_Raven/KiCad/StepperZ1234.sch (KiCad schematic (older format))
At the start: 80 parts, among them J10 CONN_01X04, J11 CONN_01X04, J8 CONN_01X04, J9 CONN_01X04, U5 TMC2130, U6 TMC2130, U7 TMC2130, U8 TMC2130

Commit message: TMC2209 upgrade layout ready for review
Parts:
- removed C59, C60, C61, C62, C63, C64, C87, C88, C89, C90, C91, C92: 100nF, MZBOT:C_0603, symbol Voron_Klipper_Board-rescue:C_0805-MZBOT
- removed R17, R18, R25, R26: 10.0K, MZBOT:R_0603, symbol Voron_Klipper_Board-rescue:R_0805-MZBOT
- removed R19, R20, R27, R28: 10R, MZBOT:R_0603, symbol Voron_Klipper_Board-rescue:R_0805-MZBOT
- removed U5, U6, U7, U8: TMC2130, MZBOT:QFN36_0.5_5.0X6.0, symbol Voron_Klipper_Board-rescue:TMC2130-MZBOT
- added C33, C35, C59, C60: 100nF, MZBOT:C_0603, symbol MZBOT:C_0805
- added C34, C36, C61, C62: 4.7uF, MZBOT:C_0805, symbol MZBOT:C_0805
- added R10, R4, R9: 10.0K, MZBOT:R_0603, symbol MZBOT:R_0805
- added U5, U6, U7, U8: TMC2209, MZBOT:QFN-28_EP_5x5_Pitch0.5mm, symbol MZBOT:TMC2209
- C100, C101, C102, C103, C104, C105, C106, C108, C110, C111, C112, C57, C58, C65, C66, C67, C68, C69, C70, C71, C72, C73, C74, C75, C76, C77, C78, C80, C82, C83, C84, C85, C86, C93, C94, C95, C96, C97, C98, C99: symbol Voron_Klipper_Board-rescue:C_0805-MZBOT -> MZBOT:C_0805
- C107, C109, C79, C81: symbol Voron_Klipper_Board-rescue:CP1-MZBOT -> MZBOT:CP1
- J10, J11, J8, J9: symbol Voron_Klipper_Board-rescue:CONN_01X04-MZBOT -> MZBOT:CONN_01X04
- R21, R22, R23, R24, R29, R30, R31, R32: symbol Voron_Klipper_Board-rescue:R_0805-MZBOT -> MZBOT:R_0805
Connections:
- net labels added: TMC_UART1
- net labels removed: +5V, SPI_CLK, SPI_CS_Z0, SPI_CS_Z1, SPI_CS_Z2, SPI_CS_Z3, SPI_SDI, SPI_SDO
- wire segments 512 -> 365
- no-connect marks 0 -> 12
