File: Taco_Raven/KiCad/Thermistors.sch (KiCad schematic (older format))
At the start: 20 parts, among them J20 CONN_01X02, J21 CONN_01X02, J22 CONN_01X02, J23 CONN_01X02, J24 CONN_01X02

Commit message: TMC2209 upgrade layout ready for review
Parts:
- C129, C130, C131, C132, C133: symbol Voron_Klipper_Board-rescue:C_0805-MZBOT -> MZBOT:C_0805
- J20, J21, J22, J23, J24: symbol Voron_Klipper_Board-rescue:CONN_01X02-MZBOT -> MZBOT:CONN_01X02
- R43, R44, R45, R46, R47, R48, R49, R50, R51, R52: symbol Voron_Klipper_Board-rescue:R_0805-MZBOT -> MZBOT:R_0805
Changed lines of the file:
@@
 Connection ~ 3500 2525
 $Comp
-L Voron_Klipper_Board-rescue:GND-MZBOT #PWR?
+L MZBOT:GND #PWR?
 U 1 1 5BBA1A6F
 P 3500 2975
@@
 Connection ~ 5375 2525
 $Comp
-L Voron_Klipper_Board-rescue:GND-MZBOT #PWR?
+L MZBOT:GND #PWR?
 U 1 1 5BBB3E2A
 P 5375 2975
@@
 Connection ~ 7250 2525
 $Comp
-L Voron_Klipper_Board-rescue:GND-MZBOT #PWR?
+L MZBOT:GND #PWR?
 U 1 1 5BBB4642
 P 7250 2975
@@
 Connection ~ 3500 4250
 $Comp
-L Voron_Klipper_Board-rescue:GND-MZBOT #PWR?
+L MZBOT:GND #PWR?
 U 1 1 5BBB4AF2
 P 3500 4700
@@
 Connection ~ 5375 4250
 $Comp
-L Voron_Klipper_Board-rescue:GND-MZBOT #PWR?
+L MZBOT:GND #PWR?
 U 1 1 5BBB6119
 P 5375 4700
@@
 Text Notes 5275 5200 0    118  ~ 24
 THERMISTOR 3\n
+Text GLabel 7075 2525 0    39   Input ~ 0
+T0
 Text GLabel 3325 2525 0    39   Input ~ 0
-T0
-Text GLabel 7075 2525 0    39   Input ~ 0
 T4
-Text GLabel 3325 4250 0    39   Input ~ 0
+Text GLabel 5200 4250 0    39   Input ~ 0
 T1
 Text GLabel 5200 2525 0    39   Input ~ 0
 T2
-Text GLabel 5200 4250 0    39   Input ~ 0
+Text GLabel 3325 4250 0    39   Input ~ 0
 T3
 Text GLabel 3800 2125 0    39   Input ~ 0
@@
 VREF
 $Comp
-L Voron_Klipper_Board-rescue:CONN_01X02-MZBOT J?
+L MZBOT:CONN_01X02 J?
 U 1 1 607FFB66
 P 4500 2575
@@
 $EndComp
 $Comp
-L Voron_Klipper_Board-rescue:CONN_01X02-MZBOT J?
+L MZBOT:CONN_01X02 J?
 U 1 1 607FFC5D
 P 6375 2575
@@
 $EndComp
 $Comp
-L Voron_Klipper_Board-rescue:CONN_01X02-MZBOT J?
+L MZBOT:CONN_01X02 J?
 U 1 1 607FFCE9
 P 8250 2575
@@
 $EndComp
 $Comp
-L Voron_Klipper_Board-rescue:CONN_01X02-MZBOT J?
+L MZBOT:CONN_01X02 J?
 U 1 1 607FFD4F
 P 6375 4300
@@
 $EndComp
 $Comp
-L Voron_Klipper_Board-rescue:R_0805-MZBOT R?
+L MZBOT:R_0805 R?
 U 1 1 60806034
 P 7775 2325
@@
 $EndComp
 $Comp
-L Voron_Klipper_Board-rescue:R_0805-MZBOT R?
+L MZBOT:R_0805 R?
 U 1 1 6080A992
 P 5900 2325
@@
 $EndComp
 $Comp
-L Voron_Klipper_Board-rescue:R_0805-MZBOT R?
+L MZBOT:R_0805 R?
 U 1 1 6080AA50
 P 4025 2325
@@
 $EndComp
 $Comp
-L Voron_Klipper_Board-rescue:R_0805-MZBOT R?
+L MZBOT:R_0805 R?
 U 1 1 6080AABC
 P 4025 4050
@@
 $EndComp
 $Comp
-L Voron_Klipper_Board-rescue:R_0805-MZBOT R?
+L MZBOT:R_0805 R?
 U 1 1 6080AB62
 P 5900 4050
@@
 $EndComp
 $Comp
-L Voron_Klipper_Board-rescue:C_0805-MZBOT C?
+L MZBOT:C_0805 C?
 U 1 1 6080C862
 P 3500 2775
@@
 $EndComp
 $Comp
-L Voron_Klipper_Board-rescue:C_0805-MZBOT C?
+L MZBOT:C_0805 C?
 U 1 1 6080DE5A
 P 5375 2775
@@
 $EndComp
 $Comp
-L Voron_Klipper_Board-rescue:C_0805-MZBOT C?
+L MZBOT:C_0805 C?
 U 1 1 6080DFDD
 P 7250 2775
@@
 $EndComp
 $Comp
-L Voron_Klipper_Board-rescue:C_0805-MZBOT C?
+L MZBOT:C_0805 C?
 U 1 1 6080E2D3
 P 5375 4500
@@
 $EndComp
 $Comp
-L Voron_Klipper_Board-rescue:C_0805-MZBOT C?
+L MZBOT:C_0805 C?
 U 1 1 6080E3A8
 P 3500 4500
@@
 $EndComp
 $Comp
-L Voron_Klipper_Board-rescue:CONN_01X02-MZBOT J?
+L MZBOT:CONN_01X02 J?
 U 1 1 607FFDB5
 P 4500 4300
@@
 $EndComp
 $Comp
-L Voron_Klipper_Board-rescue:GND-MZBOT #PWR?
+L MZBOT:GND #PWR?
 U 1 1 5E8E1F49
 P 6075 4475
@@
 Connection ~ 4025 4250
 $Comp
-L Voron_Klipper_Board-rescue:GND-MZBOT #PWR?
+L MZBOT:GND #PWR?
 U 1 1 5E8E5EFB
 P 4200 4475
@@
 	4200 4350 4300 4350
 $Comp
-L Voron_Klipper_Board-rescue:GND-MZBOT #PWR?
+L MZBOT:GND #PWR?
 U 1 1 5E8E6C60
 P 4200 2750
@@
 Connection ~ 4025 2525
 $Comp
-L Voron_Klipper_Board-rescue:GND-MZBOT #PWR?
+L MZBOT:GND #PWR?
 U 1 1 5E8E89D1
 P 6075 2750
@@
 Connection ~ 5900 2525
 $Comp
-L Voron_Klipper_Board-rescue:GND-MZBOT #PWR?
+L MZBOT:GND #PWR?
 U 1 1 5E8EA414
 P 7950 2750
@@
 Changed J20,21,22,23,24 to be low side connected\nChanged R43,44,47,48,51 from 10 to 1K\n\n
 $Comp
-L Voron_Klipper_Board-rescue:R_0805-MZBOT R?
+L MZBOT:R_0805 R?
 U 1 1 5E9C865D
 P 3775 2525
@@
 $EndComp
 $Comp
-L Voron_Klipper_Board-rescue:R_0805-MZBOT R?
+L MZBOT:R_0805 R?
 U 1 1 5E9CFB78
 P 5650 2525
@@
 $EndComp
 $Comp
-L Voron_Klipper_Board-rescue:R_0805-MZBOT R?
+L MZBOT:R_0805 R?
 U 1 1 5E9D1A9A
 P 5650 4250
@@
 $EndComp
 $Comp
-L Voron_Klipper_Board-rescue:R_0805-MZBOT R?
+L MZBOT:R_0805 R?
 U 1 1 5E9D2A61
 P 3775 4250
@@
 $EndComp
 $Comp
-L Voron_Klipper_Board-rescue:R_0805-MZBOT R?
+L MZBOT:R_0805 R?
 U 1 1 5E9D0C37
 P 7525 2525
