File: Taco_Raven/KiCad/Voron_Klipper_Board.sch (KiCad schematic (older format))
At the start: 9 parts

Commit message: TMC2209 upgrade layout ready for review
Parts:
- FID1, FID2, FID3: symbol Voron_Klipper_Board-rescue:FIDUCIAL_1MM-MZBOT -> MZBOT:FIDUCIAL_1MM
- G1: symbol Voron_Klipper_Board-rescue:TACo-MZBOT -> MZBOT:TACo
- G2: symbol Voron_Klipper_Board-rescue:mzbot-MZBOT -> MZBOT:mzbot
- MH1, MH2, MH3, MH4: symbol Voron_Klipper_Board-rescue:MountingHole-MZBOT -> MZBOT:MountingHole
Changed lines of the file:
@@
 $EndSheet
 $Comp
-L Voron_Klipper_Board-rescue:FIDUCIAL_1MM-MZBOT FID1
+L MZBOT:FIDUCIAL_1MM FID1
 U 1 1 5CADE6A5
 P 5950 4950
@@
 $EndComp
 $Comp
-L Voron_Klipper_Board-rescue:FIDUCIAL_1MM-MZBOT FID2
+L MZBOT:FIDUCIAL_1MM FID2
 U 1 1 5CADE6C7
 P 6225 4950
@@
 $EndComp
 $Comp
-L Voron_Klipper_Board-rescue:FIDUCIAL_1MM-MZBOT FID3
+L MZBOT:FIDUCIAL_1MM FID3
 U 1 1 5CADE6E9
 P 6500 4950
@@
 $EndComp
 $Comp
-L Voron_Klipper_Board-rescue:MountingHole-MZBOT MH1
+L MZBOT:MountingHole MH1
 U 1 1 5CADE712
 P 5950 5175
@@
 $EndComp
 $Comp
-L Voron_Klipper_Board-rescue:MountingHole-MZBOT MH2
+L MZBOT:MountingHole MH2
 U 1 1 5CADE7C5
 P 6225 5175
@@
 $EndComp
 $Comp
-L Voron_Klipper_Board-rescue:MountingHole-MZBOT MH3
+L MZBOT:MountingHole MH3
 U 1 1 5CADE871
 P 6500 5175
@@
 $EndComp
 $Comp
-L Voron_Klipper_Board-rescue:TACo-MZBOT G1
+L MZBOT:TACo G1
 U 1 1 60A4986D
 P 7425 5125
@@
 $EndComp
 $Comp
-L Voron_Klipper_Board-rescue:mzbot-MZBOT G2
+L MZBOT:mzbot G2
 U 1 1 60A4A39C
 P 8025 5150
@@
 $EndComp
 $Comp
-L Voron_Klipper_Board-rescue:MountingHole-MZBOT MH4
+L MZBOT:MountingHole MH4
 U 1 1 60A4B4FD
 P 6775 5175
